File: mult.kicad_pcb (KiCad board)
At the start: 2 copper layers, 55.5 x 89.7 mm, 47 parts, among them J1 Conn_02x05_Odd_Even, J10 Conn_01x03_Pin, J11 Conn_01x03_Pin, J12 Conn_01x03_Pin, J13 Conn_01x03_Socket, J14 Conn_01x03_Socket, J15 Conn_01x03_Socket, J2 AudioJack2_SwitchT, J3 AudioJack2_SwitchT, J4 AudioJack2_SwitchT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

Commit message: Bugfixes from v0
Parts:
- removed the R3 at (136.4, 69.5)
- removed the R4 at (136.4, 73.3)
- removed the R8 at (149.7, 85.4)
- removed R9: 100K, Resistor_SMD:R_0805_2012Metric
- U2: value TL074 -> TL072; footprint Package_SO:SOIC-14_3.9x8.7mm_P1.27mm -> Package_SO:SOIC-8_3.9x4.9mm_P1.27mm
- moved R6 15.0 mm to (150.4, 80.0), turned to 0 degrees
- moved C3 13.6 mm to (136.1, 72.4)
- moved R5 11.7 mm to (150.4, 74.9), turned to 0 degrees
- moved R7 10.2 mm to (150.4, 82.3), turned to 0 degrees
- moved R8 7.20 mm to (150.4, 84.6), turned to 0 degrees
- moved R4 5.86 mm to (150.4, 72.4), turned to 0 degrees
- moved C4 3.34 mm to (139.7, 82.0)
- moved U2 2.34 mm to (144.8, 82.3), turned to -90 degrees
- moved U1 1.27 mm to (143.4, 72.7)
- moved R3 0.72 mm to (150.4, 69.8), turned to 0 degrees
- renumbered R5 to R3, R6 to R4, R7 to R5, R10 to R6, R11 to R7, R12 to R8
Connections:
- R3 pad 1: Net-(U1B--) -> Net-(U1A--)
- R4 pad 1: Net-(U1C--) -> Net-(U1B--)
- R5 pad 1: Net-(U1D--) -> Net-(U1C--)
- R6 pad 1: Net-(U2B--) -> Net-(U1D--)
- R7 pad 1: Net-(U2C--) -> Net-(U2A--)
- R8 pad 1: Net-(U2D--) -> Net-(U2B--)
- U1 pad 1: Net-(U1B-+) -> Net-(U1A--)
- U1 pad 10: Net-(U1B-+) -> /IN0'
- U1 pad 12: Net-(U1B-+) -> /IN1'
- U1 pad 2: GND -> Net-(U1A--)
- U1 pad 3: Net-(U1A-+) -> /IN0'
- U1 pad 5: Net-(U1B-+) -> /IN0'
- U2 pad 1: Net-(U2B-+) -> Net-(U2A--)
- U2 pad 2: GND -> Net-(U2A--)
- U2 pad 3: Net-(U2A-+) -> /IN1'
- U2 pad 4: +12V -> -12V
- U2 pad 5: Net-(U2B-+) -> /IN1'
- U2 pad 8: Net-(U2C--) -> +12V
Routing:
- net Net-(U2B-+): track 22.1 -> 0.00 mm, vias 2 -> 0
- net Net-(U1B-+): track 21.8 -> 0.00 mm, vias 3 -> 0
- net /OUT3': track 25.3 -> 6.73 mm, vias 1 -> 0
- net /IN0': track 36.3 -> 51.6 mm
- net /OUT4': track 21.7 -> 6.83 mm
- net /IN1': track 47.5 -> 61.6 mm
- net /OUT2': track 20.5 -> 6.73 mm, vias 1 -> 0
- net Net-(U2A--): track 0.00 -> 13.5 mm, vias 0 -> 2
- net Net-(U1A--): track 0.00 -> 12.6 mm
- net Net-(U1A-+): track 11.5 -> 0.00 mm
- net Net-(U1D--): track 4.12 -> 14.7 mm
- net +12V: track 68.8 -> 58.8 mm
- net Net-(U2A-+): track 9.48 -> 0.00 mm, vias 2 -> 0
- net /OUT5': track 16.1 -> 6.94 mm
- net /OUT1': track 14.5 -> 6.73 mm
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Other:
- board text added: "thismatters/mult/v1"
- board text removed: "thismatters/mult/v0"

Commit message: prepping v1
Parts:
- added H13: Standoff, MountingHole:MountingHole_2.7mm_M2.5, B.Cu at (159.1, 77.5)
- added H14: Standoff, MountingHole:MountingHole_2.7mm_M2.5, F.Cu at (105.1, 85.1)
- added H15: Standoff, MountingHole:MountingHole_2.7mm_M2.5, F.Cu at (159.1, 102.5)
- added H16: Standoff, MountingHole:MountingHole_2.7mm_M2.5, F.Cu at (105.1, 110.1)
- C3, C4, D1, D2, R1, R2, R3, R4, R5, R6, R7, R8, U1, U2: moved to F.Cu
- moved C2 17.6 mm to (123.6, 69.6), turned to 180 degrees
- moved D1 5.22 mm to (119.4, 72.6), turned to -90 degrees
- moved D2 4.91 mm to (119.4, 82.3), turned to -90 degrees
- moved R2 4.12 mm to (119.4, 76.2)
- moved R1 4.12 mm to (119.4, 78.7)
- moved H1 2.53 mm to (106.8, 119.3)
- moved H2 2.53 mm to (157.4, 119.3)
- moved H4 2.53 mm to (106.8, 152.9)
- moved H3 2.52 mm to (157.6, 152.9)
- moved C1 1.98 mm to (121.2, 85.2), turned to 0 degrees
- moved J12 0.44 mm to (157.4, 106.7)
- moved J15 0.44 mm to (157.4, 81.7)
- moved J11 0.44 mm to (157.5, 93.2)
- moved J14 0.44 mm to (157.5, 68.1)
- turned C3 to 90 degrees
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Connections:
- R3 pad 1: Net-(U1A--) -> Net-(U1D--)
- R4 pad 1: Net-(U1B--) -> Net-(U1C--)
- R5 pad 1: Net-(U1C--) -> Net-(U1B--)
- R6 pad 1: Net-(U1D--) -> Net-(U1A--)
- R7 pad 1: Net-(U2A--) -> Net-(U2B--)
- R8 pad 1: Net-(U2B--) -> Net-(U2A--)
- U1 pad 12: /IN1' -> /IN0'
- U1 pad 3: /IN0' -> /IN1'
Routing:
- net GND: track 0.00 -> 123.3 mm, vias 0 -> 1
- net Net-(U2A--): track 13.5 -> 8.68 mm, vias 2 -> 0
- net Net-(J1-Pin_10): track 11.8 -> 7.80 mm
- net Net-(U1D--): track 14.7 -> 11.8 mm
- net Net-(D2-COM): track 2.52 -> 4.87 mm
- net -12V: track 58.8 -> 60.9 mm
- net +12V: track 58.8 -> 57.3 mm
- net Net-(D1-COM): track 4.39 -> 3.00 mm
- net Net-(U1B--): track 4.43 -> 3.29 mm
- net /OUT1: track 21.2 -> 22.2 mm
- net Net-(J1-Pin_1): track 8.21 -> 7.26 mm
- net Net-(U1C--): track 3.63 -> 4.43 mm
- net /OUT4: track 31.0 -> 30.2 mm
- net /OUT3: track 42.4 -> 41.9 mm
- net /OUT5: track 6.73 -> 6.22 mm
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Other:
- board size 55.5 x 89.7 mm -> 60.6 x 89.7 mm
- board text removed: "POWER"
