File: mult.kicad_sch (KiCad schematic)
At the start: 47 parts, among them J1 Conn_02x05_Odd_Even, J10 Conn_01x03_Pin, J11 Conn_01x03_Pin, J12 Conn_01x03_Pin, J13 Conn_01x03_Socket, J14 Conn_01x03_Socket, J15 Conn_01x03_Socket, J2 AudioJack2_SwitchT, J3 AudioJack2_SwitchT, J4 AudioJack2_SwitchT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

Commit message: forgot to hit save
Parts:
- U1, U2: PartNum (none) -> 595-TL074CDR; Vendor (none) -> Mouser
Changed lines of the file:
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@@
+      (effects (font (size 1.27 1.27)) hide)
+    )
+    (property "Vendor" "Mouser" (at 214.63 66.04 0)
+      (effects (font (size 1.27 1.27)) hide)
+    )
+    (property "PartNum" "595-TL074CDR" (at 214.63 66.04 0)
       (effects (font (size 1.27 1.27)) hide)
     )
@@
     )
     (property "Datasheet" "http://www.ti.com/lit/ds/symlink/tl071.pdf" (at 134.62 43.18 0)
+      (effects (font (size 1.27 1.27)) hide)
+    )
+    (property "Vendor" "Mouser" (at 133.35 48.26 0)
+      (effects (font (size 1.27 1.27)) hide)
+    )
+    (property "PartNum" "595-TL074CDR" (at 133.35 48.26 0)
       (effects (font (size 1.27 1.27)) hide)
     )
@@
       (effects (font (size 1.27 1.27)) hide)
     )
+    (property "Vendor" "Mouser" (at 101.6 43.18 0)
+      (effects (font (size 1.27 1.27)) hide)
+    )
+    (property "PartNum" "595-TL074CDR" (at 101.6 43.18 0)
+      (effects (font (size 1.27 1.27)) hide)
+    )
     (pin "14")
     (pin "3")
@@
       (effects (font (size 1.27 1.27)) hide)
     )
+    (property "Vendor" "Mouser" (at 246.38 149.86 0)
+      (effects (font (size 1.27 1.27)) hide)
+    )
+    (property "PartNum" "595-TL074CDR" (at 246.38 149.86 0)
+      (effects (font (size 1.27 1.27)) hide)
+    )
     (pin "8")
     (pin "4")
@@
     )
     (property "Datasheet" "http://www.ti.com/lit/ds/symlink/tl071.pdf" (at 181.61 43.18 0)
+      (effects (font (size 1.27 1.27)) hide)
+    )
+    (property "Vendor" "Mouser" (at 180.34 48.26 0)
+      (effects (font (size 1.27 1.27)) hide)
+    )
+    (property "PartNum" "595-TL074CDR" (at 180.34 48.26 0)
       (effects (font (size 1.27 1.27)) hide)
     )
@@
       (effects (font (size 1.27 1.27)) hide)
     )
+    (property "Vendor" "Mouser" (at 214.63 30.48 0)
+      (effects (font (size 1.27 1.27)) hide)
+    )
+    (property "PartNum" "595-TL074CDR" (at 214.63 30.48 0)
+      (effects (font (size 1.27 1.27)) hide)
+    )
     (pin "8")
     (pin "4")
@@
     )
     (property "Datasheet" "http://www.ti.com/lit/ds/symlink/tl071.pdf" (at 134.62 60.96 0)
+      (effects (font (size 1.27 1.27)) hide)
+    )
+    (property "Vendor" "Mouser" (at 133.35 66.04 0)
+      (effects (font (size 1.27 1.27)) hide)
+    )
+    (property "PartNum" "595-TL074CDR" (at 133.35 66.04 0)
       (effects (font (size 1.27 1.27)) hide)
     )
@@
       (effects (font (size 1.27 1.27)) hide)
     )
+    (property "Vendor" "Mouser" (at 133.35 30.48 0)
+      (effects (font (size 1.27 1.27)) hide)
+    )
+    (property "PartNum" "595-TL074CDR" (at 133.35 30.48 0)
+      (effects (font (size 1.27 1.27)) hide)
+    )
     (pin "14")
     (pin "3")
@@
       (effects (font (size 1.27 1.27)) hide)
     )
+    (property "Vendor" "Mouser" (at 214.63 48.26 0)
+      (effects (font (size 1.27 1.27)) hide)
+    )
+    (property "PartNum" "595-TL074CDR" (at 214.63 48.26 0)
+      (effects (font (size 1.27 1.27)) hide)
+    )
     (pin "8")
     (pin "4")
@@
       (effects (font (size 1.27 1.27)) hide)
     )
+    (property "Vendor" "Mouser" (at 212.09 149.86 0)
+      (effects (font (size 1.27 1.27)) hide)
+    )
+    (property "PartNum" "595-TL074CDR" (at 212.09 149.86 0)
+      (effects (font (size 1.27 1.27)) hide)
+    )

Commit message: Bugfixes from v0
Parts:
- removed R3, R4, R8, R9: 100K, Resistor_SMD:R_0805_2012Metric, symbol Device:R
- removed U2: TL074, Package_SO:SOIC-14_3.9x8.7mm_P1.27mm, symbol Amplifier_Operational:TL074
- added U2: TL072, Package_SO:SOIC-8_3.9x4.9mm_P1.27mm, symbol Amplifier_Operational:TL072
- renumbered R5 to R3, R6 to R4, R7 to R5, R10 to R6, R11 to R7, R12 to R8
Connections:
- net +12V: now also U2.8 (V+)
- net -12V: now also U2.4 (V-)
- net GND: no longer U1.2 (-)
- net IN0': now also U1.10 (+), U1.3 (+), U1.5 (+)
- net IN1': now also U1.12 (+), U2.3 (+), U2.5 (+)
- net at R8.1: now also U2.6 (-), U2.7
- net at U1.8, U1.9 (-): now also R5.1; no longer R4.1
- net at R6.1: now also U1.13 (-), U1.14
- net at R7.1: now also U2.1, U2.2 (-)
- net at U1.6 (-), U1.7: now also R4.1; no longer R3.1
- new net: R3.1, U1.1, U1.2 (-)
Other:
- moved on the sheet: R3, R4, R5, U1A, U1B, U1C, U1D

Commit message: prepping v1
Parts:
- added H13, H14, H15, H16: Standoff, MountingHole:MountingHole_2.7mm_M2.5, symbol Mechanical:MountingHole
- added M1, M2: Standoff, Eurorack:Standoff_M2.5x0.45-11mm, symbol Eurorack:Standoff
- added M3, M4, M5, M6: Screw, Eurorack:Screw_M2.5x0.45-6mm, symbol Eurorack:Screw
Connections:
- net IN0': now also U1.12 (+); no longer U1.3 (+)
- net IN1': now also U1.3 (+); no longer U1.12 (+)
- net at U2.6 (-), U2.7: now also R7.1; no longer R8.1
- net at U1.8, U1.9 (-): now also R4.1; no longer R5.1
- net at U1.1, U1.2 (-): now also R6.1; no longer R3.1
- net at U1.13 (-), U1.14: now also R3.1; no longer R6.1
- net at U1.6 (-), U1.7: now also R5.1; no longer R4.1
- net at U2.1, U2.2 (-): now also R8.1; no longer R7.1
Other:
- note added: "Mechanical attachment for 3 layer module"
- moved on the sheet: U1A, U1B, U1C, U1D, U2A, U2B
